File: Hardware/Console_Block.sch (EAGLE design)
At the start: 39 parts, among them Q1 BSS138, U2 FTS31XS-U, U4 TPS62065

Commit message: Ready for reds Tweaked silk positions, add some restrict between pads on QFN No known to-do items
Parts:
- U2: value FTS31XS-U -> FT231XS-U
Changed lines of the file:
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@@
 <part name="GND1" library="SparkFun-Aesthetics" deviceset="GND" device=""/>
 <part name="GND5" library="SparkFun-Aesthetics" deviceset="GND" device=""/>
-<part name="U2" library="SparkFun-DigitalIC" deviceset="FT231X" device="S" value="FTS31XS-U"/>
+<part name="U2" library="SparkFun-DigitalIC" deviceset="FT231X" device="S" value="FT231XS-U"/>
 <part name="C1" library="SparkFun-Capacitors" deviceset="0.1UF-25V-5%(0603)" device="" value="0.1uF"/>
 <part name="C2" library="SparkFun-Capacitors" deviceset="0.1UF-25V-5%(0603)" device="" value="0.1uF"/>
@@
 <instance part="JP1" gate="G$1" x="27.94" y="137.16" rot="MR0"/>
 <instance part="GND1" gate="1" x="38.1" y="121.92" rot="MR0"/>
-<instance part="GND5" gate="1" x="17.78" y="137.16" rot="MR90"/>
+<instance part="GND5" gate="1" x="17.78" y="132.08" rot="MR0"/>
 <instance part="U2" gate="G$1" x="86.36" y="134.62"/>
 <instance part="C1" gate="G$1" x="81.28" y="170.18" rot="R180"/>
@@
 <pinref part="JP1" gate="G$1" pin="SHIELD"/>
 <pinref part="GND5" gate="1" pin="GND"/>
+<wire x1="17.78" y1="134.62" x2="17.78" y2="137.16" width="0.1524" layer="91"/>
+<wire x1="17.78" y1="137.16" x2="20.32" y2="137.16" width="0.1524" layer="91"/>
 </segment>
 <segment>

Commit message: added bottom side fiducials
Parts:
- added FID3, FID4: FIDUCIAL1X2, SparkFun-Aesthetics:FIDUCIAL1X2
Changed lines of the file:
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@@
 <part name="R10" library="SparkFun-Resistors" deviceset="1KOHM1/10W1%(0603)" device="" value="1K"/>
 <part name="SUPPLY7" library="SparkFun-Aesthetics" deviceset="5V" device=""/>
+<part name="FID3" library="SparkFun-Aesthetics" deviceset="FIDUCIAL" device="1X2"/>
+<part name="FID4" library="SparkFun-Aesthetics" deviceset="FIDUCIAL" device="1X2"/>
 </parts>
 <sheets>
@@
 <instance part="R10" gate="G$1" x="185.42" y="76.2" rot="R180"/>
 <instance part="SUPPLY7" gate="G$1" x="177.8" y="78.74"/>
+<instance part="FID3" gate="G$1" x="238.76" y="30.48"/>
+<instance part="FID4" gate="G$1" x="243.84" y="30.48"/>
 </instances>
 <busses>
